File: ServosControl/ATmegaProgramming.sch (EAGLE design)
At the start: 5 parts, among them U1 ATMEGA88PA-MU

Commit message: Updating board
Parts:
- added BUS: CONNEC_1X03, RobotCampus:CONNEC_1X03
- added C1: 100nF, rhoban:C_EU-100NF
- R1: device resistor:R-EU_0414/15 -> rhoban:RESISTANCE-R0805
- renumbered U$1 to RESONATOR, U$2 to ISP1, U$3 to ISP2
Connections:
- net DATA: now also BUS.3
- net GND: now also BUS.2, C1.2
- net VCC: now also BUS.1, C1.1
Changed lines of the file:
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@@
 </classes>
 <parts>
-<part name="U1" library="RobotCampus" deviceset="ATMEGA88PA-MU" device=""/>
+<part name="U1" library="RobotCampus" deviceset="ATMEGA88PA-MU" device="" value=""/>
 <part name="P+1" library="supply1" deviceset="VCC" device=""/>
 <part name="GND1" library="supply1" deviceset="GND" device=""/>
-<part name="U$1" library="RobotCampus" deviceset="SG-310" device=""/>
+<part name="RESONATOR" library="RobotCampus" deviceset="SG-310" device=""/>
 <part name="P+4" library="supply1" deviceset="VCC" device=""/>
 <part name="GND4" library="supply1" deviceset="GND" device=""/>
-<part name="U$2" library="RobotCampus" deviceset="CONNEC_1X03" device=""/>
-<part name="U$3" library="RobotCampus" deviceset="CONNEC_1X03" device=""/>
+<part name="ISP1" library="RobotCampus" deviceset="CONNEC_1X03" device=""/>
+<part name="ISP2" library="RobotCampus" deviceset="CONNEC_1X03" device=""/>
 <part name="P+2" library="supply1" deviceset="VCC" device=""/>
 <part name="GND2" library="supply1" deviceset="GND" device=""/>
 <part name="P+3" library="supply1" deviceset="VCC" device=""/>
-<part name="R1" library="resistor" deviceset="R-EU_" device="0414/15"/>
+<part name="BUS" library="RobotCampus" deviceset="CONNEC_1X03" device=""/>
+<part name="P+5" library="supply1" deviceset="VCC" device=""/>
+<part name="GND3" library="supply1" deviceset="GND" device=""/>
+<part name="R1" library="rhoban" deviceset="RESISTANCE" device="-R0805"/>
+<part name="C1" library="rhoban" deviceset="C_EU" device="-100NF" value="100nF"/>
+<part name="P+6" library="supply1" deviceset="VCC" device=""/>
+<part name="GND5" library="supply1" deviceset="GND" device=""/>
 </parts>
 <sheets>
@@
 <instance part="U1" gate="A" x="30.48" y="55.88"/>
 <instance part="P+1" gate="VCC" x="7.62" y="83.82"/>
-<instance part="GND1" gate="1" x="7.62" y="20.32"/>
-<instance part="U$1" gate="A" x="88.9" y="33.02"/>
+<instance part="GND1" gate="1" x="7.62" y="17.78"/>
+<instance part="RESONATOR" gate="A" x="88.9" y="33.02"/>
 <instance part="P+4" gate="VCC" x="73.66" y="43.18"/>
 <instance part="GND4" gate="1" x="73.66" y="30.48"/>
-<instance part="U$2" gate="G$1" x="-30.48" y="73.66"/>
-<instance part="U$3" gate="G$1" x="-30.48" y="58.42"/>
+<instance part="ISP1" gate="G$1" x="-30.48" y="73.66"/>
+<instance part="ISP2" gate="G$1" x="-30.48" y="58.42"/>
 <instance part="P+2" gate="VCC" x="-33.02" y="66.04"/>
 <instance part="GND2" gate="1" x="-33.02" y="55.88"/>
 <instance part="P+3" gate="VCC" x="-2.54" y="53.34"/>
+<instance part="BUS" gate="G$1" x="-40.64" y="27.94"/>
+<instance part="P+5" gate="VCC" x="-45.72" y="38.1"/>
+<instance part="GND3" gate="1" x="-50.8" y="30.48" rot="R270"/>
 <instance part="R1" gate="G$1" x="-2.54" y="45.72" rot="R90"/>
+<instance part="C1" gate="G$1" x="-12.7" y="25.4"/>
+<instance part="P+6" gate="VCC" x="-12.7" y="33.02"/>
+<instance part="GND5" gate="1" x="-12.7" y="20.32"/>
 </instances>
 <busses>
@@
 </segment>
 <segment>
-<pinref part="U$1" gate="A" pin="VCC"/>
+<pinref part="RESONATOR" gate="A" pin="VCC"/>
 <pinref part="P+4" gate="VCC" pin="VCC"/>
 </segment>
 <segment>
-<pinref part="U$3" gate="G$1" pin="1"/>
+<pinref part="ISP2" gate="G$1" pin="1"/>
 <wire x1="-27.94" y1="63.5" x2="-33.02" y2="63.5" width="0.1524" layer="91"/>
 <pinref part="P+2" gate="VCC" pin="VCC"/>
 </segment>
 <segment>
+<pinref part="BUS" gate="G$1" pin="1"/>
+<pinref part="P+5" gate="VCC" pin="VCC"/>
+<wire x1="-38.1" y1="33.02" x2="-45.72" y2="33.02" width="0.1524" layer="91"/>
+<wire x1="-45.72" y1="33.02" x2="-45.72" y2="35.56" width="0.1524" layer="91"/>
+</segment>
+<segment>
 <pinref part="P+3" gate="VCC" pin="VCC"/>
 <pinref part="R1" gate="G$1" pin="2"/>
+</segment>
+<segment>
+<pinref part="C1" gate="G$1" pin="1"/>
+<pinref part="P+6" gate="VCC" pin="VCC"/>
 </segment>
 </net>
@@
 <pinref part="U1" gate="A" pin="GND_3"/>
 <wire x1="7.62" y1="27.94" x2="7.62" y2="25.4" width="0.1524" layer="91"/>
-<wire x1="7.62" y1="25.4" x2="7.62" y2="22.86" width="0.1524" layer="91"/>
+<wire x1="7.62" y1="25.4" x2="7.62" y2="20.32" width="0.1524" layer="91"/>
 <wire x1="12.7" y1="27.94" x2="7.62" y2="27.94" width="0.1524" layer="91"/>
 <pinref part="U1" gate="A" pin="GND"/>
@@
 </segment>
 <segment>
-<pinref part="U$1" gate="A" pin="GND"/>
+<pinref part="RESONATOR" gate="A" pin="GND"/>
 <pinref part="GND4" gate="1" pin="GND"/>
 </segment>
 <segment>
-<pinref part="U$3" gate="G$1" pin="3"/>
+<pinref part="ISP2" gate="G$1" pin="3"/>
 <wire x1="-27.94" y1="58.42" x2="-33.02" y2="58.42" width="0.1524" layer="91"/>
 <pinref part="GND2" gate="1" pin="GND"/>
+</segment>
+<segment>
+<pinref part="BUS" gate="G$1" pin="2"/>
+<pinref part="GND3" gate="1" pin="GND"/>
+<wire x1="-38.1" y1="30.48" x2="-48.26" y2="30.48" width="0.1524" layer="91"/>
+</segment>
+<segment>
+<pinref part="C1" gate="G$1" pin="2"/>
+<pinref part="GND5" gate="1" pin="GND"/>
 </segment>
 </net>
@@
 <label x="55.88" y="78.74" size="1.778" layer="95"/>
 </segment>
+<segment>
+<pinref part="BUS" gate="G$1" pin="3"/>
+<wire x1="-38.1" y1="27.94" x2="-45.72" y2="27.94" width="0.1524" layer="91"/>
+<label x="-48.26" y="25.4" size="1.778" layer="95"/>
+</segment>
 </net>
 <net name="MOTORPOS" class="0">
@@
 </segment>
 <segment>
-<pinref part="U$1" gate="A" pin="OUT"/>
+<pinref part="RESONATOR" gate="A" pin="OUT"/>
 <wire x1="104.14" y1="40.64" x2="106.68" y2="40.64" width="0.1524" layer="91"/>
 <label x="109.22" y="40.64" size="1.778" layer="95"/>
@@
 <net name="MISO" class="0">
 <segment>
-<pinref part="U$2" gate="G$1" pin="1"/>
+<pinref part="ISP1" gate="G$1" pin="1"/>
 <wire x1="-27.94" y1="78.74" x2="-33.02" y2="78.74" width="0.1524" layer="91"/>
 <label x="-38.1" y="78.74" size="1.778" layer="95"/>
@@
 <net name="SCK" class="0">
 <segment>
-<pinref part="U$2" gate="G$1" pin="2"/>
+<pinref part="ISP1" gate="G$1" pin="2"/>
 <wire x1="-27.94" y1="76.2" x2="-33.02" y2="76.2" width="0.1524" layer="91"/>
 <label x="-38.1" y="76.2" size="1.778" layer="95"/>
@@
 <net name="RESET" class="0">
 <segment>
-<pinref part="U$2" gate="G$1" pin="3"/>
+<pinref part="ISP1" gate="G$1" pin="3"/>
 <wire x1="-27.94" y1="73.66" x2="-33.02" y2="73.66" width="0.1524" layer="91"/>
 <label x="-38.1" y="73.66" size="1.778" layer="95"/>
@@
 <net name="MOSI" class="0">
 <segment>
-<pinref part="U$3" gate="G$1" pin="2"/>
+<pinref part="ISP2" gate="G$1" pin="2"/>
 <wire x1="-27.94" y1="60.96" x2="-33.02" y2="60.96" width="0.1524" layer="91"/>
 <label x="-38.1" y="60.96" size="1.778" layer="95"/>
