File: ControlV3/control.sch (EAGLE design)
At the start: 42 parts, among them P1 CONNEC_1X03, P10 CONNEC_1X03, P11 CONNEC_1X03, P12 CONNEC_1X03, P2 CONNEC_1X03, P3 CONNEC_1X03, P4 CONNEC_1X03, P5 CONNEC_1X03, P6 CONNEC_1X03, P7 CONNEC_1X03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

Commit message: Adding PDF
Other:
- note added: "Diode ou jumper"
Changed lines of the file:
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@@
 <sheet>
 <plain>
+<text x="68.58" y="-15.24" size="1.778" layer="95">Diode ou jumper</text>
 </plain>
 <instances>
