File: ControlV4/control.brd (EAGLE design)
At the start: 50 x 55 mm, 55 parts, among them P1 CONNEC_1X03, P10 CONNEC_1X03, P11 CONNEC_1X03, P12 CONNEC_1X03, P2 CONNEC_1X03, P3 CONNEC_1X03, P4 CONNEC_1X03, P5 CONNEC_1X03, P6 CONNEC_1X03, P7 CONNEC_1X03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

Commit message: Fixing the 33/3.3 problem
Connections:
- removed net 33: R15.1, R16.1, XB1.1, XB1.14
- net 3.3: now also R15.1, R16.1, XB1.1, XB1.14
Routing:
- net 3.3: track 11.2 -> 99.8 mm, vias 0 -> 2
- net 33: track 68.0 -> 0.00 mm, vias 2 -> 0
Changed lines of the file:
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@@
 <via x="12.4" y="3.6" extent="1-16" drill="0.6096"/>
-</signal>
-<signal name="33">
-<contactref element="XB1" pad="1"/>
-<contactref element="XB1" pad="14"/>
-<contactref element="R15" pad="1"/>
-<contactref element="R16" pad="1"/>
-<wire x1="23.8" y1="36.2" x2="22.8" y2="35.2" width="0.254" layer="16"/>
-<wire x1="26.7" y1="36.2" x2="23.8" y2="36.2" width="0.254" layer="16"/>
-<wire x1="27.8" y1="35.1" x2="26.7" y2="36.2" width="0.254" layer="16"/>
-<wire x1="22.8" y1="35.2" x2="22.74" y2="35.13" width="0.254" layer="16"/>
-<wire x1="27.8" y1="35.1" x2="27.82" y2="35.03" width="0.254" layer="16"/>
-<wire x1="15.4" y1="7.3" x2="13.5" y2="9.2" width="0.254" layer="16"/>
-<wire x1="29.1" y1="7.3" x2="15.4" y2="7.3" width="0.254" layer="16"/>
-<wire x1="31.6" y1="9.8" x2="31.55" y2="9.75" width="0.254" layer="1"/>
-<wire x1="31.55" y1="9.75" x2="29.1" y2="7.3" width="0.254" layer="1"/>
-<wire x1="34.4" y1="9.8" x2="31.6" y2="9.8" width="0.254" layer="1"/>
-<wire x1="34.4" y1="17.6" x2="34.4" y2="9.8" width="0.254" layer="1"/>
-<wire x1="34.5" y1="17.7" x2="34.4" y2="17.6" width="0.254" layer="1"/>
-<wire x1="34.5" y1="18.7" x2="34.5" y2="17.7" width="0.254" layer="1"/>
-<wire x1="34.4" y1="18.8" x2="34.5" y2="18.7" width="0.254" layer="1"/>
-<wire x1="34.4" y1="20.2" x2="34.4" y2="18.8" width="0.254" layer="1"/>
-<wire x1="35.4" y1="21.2" x2="34.4" y2="20.2" width="0.254" layer="1"/>
-<wire x1="13.5" y1="9.2" x2="13.427840625" y2="9.2055625" width="0.254" layer="16"/>
-<wire x1="35.4" y1="21.2" x2="35.427840625" y2="21.2055625" width="0.254" layer="1"/>
-<wire x1="28.6" y1="33.3" x2="28.9" y2="33.6" width="0.254" layer="1"/>
-<wire x1="28.6" y1="12.7" x2="28.6" y2="33.3" width="0.254" layer="1"/>
-<wire x1="31.55" y1="9.75" x2="28.6" y2="12.7" width="0.254" layer="1"/>
-<wire x1="27.8" y1="34.9" x2="27.82" y2="35.03" width="0.254" layer="16"/>
-<via x="29.1" y="7.3" extent="1-16" drill="0.6096"/>
-<via x="28.9" y="33.6" extent="1-16" drill="0.6096"/>
-<wire x1="28.9" y1="33.6" x2="28.9" y2="33.95" width="0.254" layer="16"/>
-<wire x1="28.9" y1="33.95" x2="27.82" y2="35.03" width="0.254" layer="16"/>
 </signal>
 <signal name="N$1">
@@
 <wire x1="26" y1="38.1" x2="23.3104375" y2="40.7895625" width="0.254" layer="16"/>
 <wire x1="23.3104375" y1="40.7895625" x2="23.2895625" y2="40.7895625" width="0.254" layer="16"/>
+<contactref element="XB1" pad="1"/>
+<contactref element="R15" pad="1"/>
+<contactref element="R16" pad="1"/>
+<wire x1="23.8" y1="36.2" x2="22.8" y2="35.2" width="0.254" layer="16"/>
+<wire x1="26.7" y1="36.2" x2="23.8" y2="36.2" width="0.254" layer="16"/>
+<wire x1="27.8" y1="35.1" x2="26.7" y2="36.2" width="0.254" layer="16"/>
+<wire x1="22.8" y1="35.2" x2="22.74" y2="35.13" width="0.254" layer="16"/>
+<wire x1="27.8" y1="35.1" x2="27.82" y2="35.03" width="0.254" layer="16"/>
+<wire x1="27.8" y1="34.9" x2="27.82" y2="35.03" width="0.254" layer="16"/>
+<contactref element="XB1" pad="14"/>
+<wire x1="15.4" y1="7.3" x2="13.5" y2="9.2" width="0.254" layer="16"/>
+<wire x1="29.1" y1="7.3" x2="15.4" y2="7.3" width="0.254" layer="16"/>
+<wire x1="31.6" y1="9.8" x2="31.55" y2="9.75" width="0.254" layer="1"/>
+<wire x1="31.55" y1="9.75" x2="29.1" y2="7.3" width="0.254" layer="1"/>
+<wire x1="34.4" y1="9.8" x2="31.6" y2="9.8" width="0.254" layer="1"/>
+<wire x1="34.4" y1="17.6" x2="34.4" y2="9.8" width="0.254" layer="1"/>
+<wire x1="34.5" y1="17.7" x2="34.4" y2="17.6" width="0.254" layer="1"/>
+<wire x1="34.5" y1="18.7" x2="34.5" y2="17.7" width="0.254" layer="1"/>
+<wire x1="34.4" y1="18.8" x2="34.5" y2="18.7" width="0.254" layer="1"/>
+<wire x1="34.4" y1="20.2" x2="34.4" y2="18.8" width="0.254" layer="1"/>
+<wire x1="35.4" y1="21.2" x2="34.4" y2="20.2" width="0.254" layer="1"/>
+<wire x1="35.4" y1="21.2" x2="35.427840625" y2="21.2055625" width="0.254" layer="1"/>
+<wire x1="28.6" y1="33.3" x2="28.9" y2="33.6" width="0.254" layer="1"/>
+<wire x1="28.6" y1="12.7" x2="28.6" y2="33.3" width="0.254" layer="1"/>
+<wire x1="31.55" y1="9.75" x2="28.6" y2="12.7" width="0.254" layer="1"/>
+<via x="29.1" y="7.3" extent="1-16" drill="0.6096"/>
+<via x="28.9" y="33.6" extent="1-16" drill="0.6096"/>
+<wire x1="28.9" y1="33.6" x2="28.9" y2="33.95" width="0.254" layer="16"/>
+<wire x1="13.4" y1="9.2" x2="13.427840625" y2="9.2055625" width="0.254" layer="16"/>
+<wire x1="13.4" y1="9.2" x2="13.5" y2="9.2" width="0.254" layer="16"/>
+<wire x1="27.9" y1="34.9" x2="28.8" y2="34" width="0.254" layer="16"/>
+<wire x1="28.8" y1="34" x2="28.9" y2="33.6" width="0.254" layer="16"/>
+<wire x1="27.9" y1="34.9" x2="27.82" y2="35.03" width="0.254" layer="16"/>
+<wire x1="19.8" y1="37.5" x2="21.5" y2="39.2" width="0.254" layer="16"/>
+<wire x1="19.6" y1="37.5" x2="19.8" y2="37.5" width="0.254" layer="16"/>
+<wire x1="17.3" y1="35.2" x2="19.6" y2="37.5" width="0.254" layer="16"/>
+<wire x1="16.3" y1="35.2" x2="17.3" y2="35.2" width="0.254" layer="16"/>
+<wire x1="15.5" y1="34.4" x2="16.3" y2="35.2" width="0.254" layer="16"/>
+<wire x1="15.5" y1="32.7" x2="15.5" y2="34.4" width="0.254" layer="16"/>
+<wire x1="17.4" y1="32.7" x2="15.5" y2="32.7" width="0.254" layer="16"/>
+<wire x1="18.5" y1="33.8" x2="17.4" y2="32.7" width="0.254" layer="16"/>
+<wire x1="18.5" y1="34.9" x2="18.5" y2="33.8" width="0.254" layer="16"/>
+<wire x1="19.9" y1="36.3" x2="18.5" y2="34.9" width="0.254" layer="16"/>
+<wire x1="23.8" y1="36.3" x2="19.9" y2="36.3" width="0.254" layer="16"/>
+<wire x1="21.5" y1="39.2" x2="21.57" y2="39.26" width="0.254" layer="16"/>
+<wire x1="23.8" y1="36.3" x2="23.8" y2="36.2" width="0.254" layer="16"/>
 </signal>
 <signal name="N$14">
