File: OpenCMXX/opencmxx.brd (EAGLE design)
At the start: 33.8 x 56 mm, 34 parts, among them P1 CONNEC_1X03, P2 CONNEC_1X03, P3 CONNEC_1X03, P4 CONNEC_1X03, P5 CONNEC_1X03, P6 CONNEC_1X03, P7 CONNEC_1X03, P8 CONNEC_1X03

Commit message: OpenCMXX
Parts:
- added IC1: (no value), SparkFun-PowerIC:78XXL
- moved C2 18.1 mm to (16.5, 17.7), turned to 180 degrees
- moved PWM_TO_V+ 15.3 mm to (29.4, 8.70), turned to 270 degrees
Connections:
- net GND: now also IC1.GND
- net PWM+: now also IC1.OUT
- net V+: now also IC1.IN
Routing:
- net V+: track 127.1 -> 144.3 mm
- net N$2: track 28.7 -> 44.6 mm, vias 2 -> 1
- net N$9: track 40.1 -> 28.2 mm, vias 1 -> 2
- net N$11: track 33.9 -> 23.1 mm
- net N$7: track 29.0 -> 18.2 mm, vias 1 -> 0
- net N$13: track 39.8 -> 30.8 mm
- net PWM+: track 57.5 -> 65.4 mm, vias 2 -> 1
- net GND: track 183.5 -> 189.1 mm, vias 2 -> 1
- net N$5: track 29.4 -> 24.4 mm
- net CM_3.3V: track 36.6 -> 40.6 mm, vias 1 -> 0
- net PWM8: track 5.44 -> 2.44 mm, vias 1 -> 0
- net N$3: track 30.8 -> 29.0 mm
- net 3.3V: track 64.6 -> 64.8 mm, vias 0 -> 1
