File: OpenCMXX/opencmxx.sch (EAGLE design)
At the start: 34 parts, among them P1 CONNEC_1X03, P2 CONNEC_1X03, P3 CONNEC_1X03, P4 CONNEC_1X03, P5 CONNEC_1X03, P6 CONNEC_1X03, P7 CONNEC_1X03, P8 CONNEC_1X03

Commit message: OpenCMXX
Parts:
- added IC1: (no value), SparkFun-PowerIC:V_REG_78XXSIDE
Connections:
- net GND: now also IC1.GND
- net PWM+: now also IC1.OUT
- net V+: now also IC1.IN
Changed lines of the file:
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@@
 <layer number="106" name="bPlate" color="7" fill="1" visible="yes" active="yes"/>
 <layer number="107" name="Crop" color="7" fill="1" visible="yes" active="yes"/>
+<layer number="108" name="tplace-old" color="10" fill="1" visible="yes" active="yes"/>
+<layer number="109" name="ref-old" color="11" fill="1" visible="yes" active="yes"/>
 <layer number="116" name="Patch_BOT" color="9" fill="4" visible="yes" active="yes"/>
 <layer number="121" name="_tsilk" color="7" fill="1" visible="yes" active="yes"/>
@@
 <layer number="144" name="Drill_legend" color="7" fill="1" visible="yes" active="yes"/>
 <layer number="151" name="HeatSink" color="7" fill="1" visible="yes" active="yes"/>
+<layer number="199" name="Contour" color="7" fill="1" visible="yes" active="yes"/>
 <layer number="200" name="200bmp" color="1" fill="10" visible="yes" active="yes"/>
 <layer number="201" name="201bmp" color="2" fill="10" visible="yes" active="yes"/>
@@
 <class number="0" name="default" width="0" drill="0">
 </class>
-<class number="1" name="alime" width="0.508" drill="0">
+<class number="1" name="alime" width="1.016" drill="0">
 </class>
 </classes>
@@
 <part name="C2" library="SparkFun-Capacitors" deviceset="CAP_POL" device="PTH2"/>
 <part name="GND1" library="supply1" deviceset="GND" device=""/>
+<part name="IC1" library="SparkFun-PowerIC" deviceset="V_REG_78XX" device="SIDE"/>
 </parts>
 <sheets>
@@
 <instance part="C2" gate="G$1" x="40.64" y="15.24"/>
 <instance part="GND1" gate="1" x="40.64" y="5.08"/>
+<instance part="IC1" gate="G$1" x="111.76" y="20.32"/>
 </instances>
 <busses>
@@
 <pinref part="GND1" gate="1" pin="GND"/>
 </segment>
+<segment>
+<pinref part="IC1" gate="G$1" pin="GND"/>
+<wire x1="111.76" y1="12.7" x2="111.76" y2="10.16" width="0.1524" layer="91"/>
+<label x="111.76" y="5.08" size="1.778" layer="95"/>
+</segment>
 </net>
 <net name="CM_3.3V" class="0">
@@
 <label x="99.06" y="35.56" size="1.778" layer="95"/>
 </segment>
+<segment>
+<pinref part="IC1" gate="G$1" pin="IN"/>
+<wire x1="104.14" y1="20.32" x2="99.06" y2="20.32" width="0.1524" layer="91"/>
+<label x="91.44" y="20.32" size="1.778" layer="95"/>
+</segment>
 </net>
 <net name="TTL" class="0">
@@
 <label x="40.64" y="20.32" size="1.778" layer="95"/>
 </segment>
-</net>
+<segment>
+<pinref part="IC1" gate="G$1" pin="OUT"/>
+<wire x1="119.38" y1="20.32" x2="124.46" y2="20.32" width="0.1524" layer="91"/>
+<label x="127" y="20.32" size="1.778" layer="95"/>
+</segment>
+</net>
